File: drehm-fc/drehm-fc.kicad_sch (KiCad schematic)
At the start: 16 parts, among them J1 TSW-113-08-T-T-RA, J4 Conn_01x04, U1 DEV-15583

Commit message: 0402 conversion, added holes for PCBA
Parts:
- C1: footprint Capacitor_SMD:C_0201_0603Metric -> Capacitor_SMD:C_0402_1005Metric; MPN C161472 -> C1853984
- C2: footprint Capacitor_SMD:C_0201_0603Metric -> Capacitor_SMD:C_0402_1005Metric; MPN C161494 -> C106204
- C3: footprint Capacitor_SMD:C_0201_0603Metric -> Capacitor_SMD:C_0402_1005Metric; MPN C76933 -> C326606
- R1, R2: footprint Resistor_SMD:R_0201_0603Metric -> Resistor_SMD:R_0402_1005Metric; MPN C490808 -> C25744
Changed lines of the file:
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@@
 			)
 		)
-		(property "Footprint" "Capacitor_SMD:C_0201_0603Metric"
+		(property "Footprint" "Capacitor_SMD:C_0402_1005Metric"
 			(at 264.16 70.1548 0)
 			(effects
@@
 			)
 		)
-		(property "MPN" "C161472"
+		(property "MPN" "C1853984"
 			(at 260.35 71.12 0)
 			(effects
@@
 		)
 		(instances
-			(project ""
+			(project "drehm-fc"
 				(path "/78677983-3e2d-46c3-90bf-4f512dd2e99e"
 					(reference "#PWR03")
@@
 			)
 		)
-		(property "Footprint" "Resistor_SMD:R_0201_0603Metric"
+		(property "Footprint" "Resistor_SMD:R_0402_1005Metric"
 			(at 144.272 74.93 90)
 			(effects
@@
 			)
 		)
-		(property "MPN" "C490808"
+		(property "MPN" "C25744"
 			(at 146.05 74.93 0)
 			(effects
@@
 		)
 		(instances
-			(project ""
+			(project "drehm-fc"
 				(path "/78677983-3e2d-46c3-90bf-4f512dd2e99e"
 					(reference "#PWR013")
@@
 		)
 		(instances
-			(project ""
+			(project "drehm-fc"
 				(path "/78677983-3e2d-46c3-90bf-4f512dd2e99e"
 					(reference "#FLG01")
@@
 			)
 		)
-		(property "Footprint" "Capacitor_SMD:C_0201_0603Metric"
+		(property "Footprint" "Capacitor_SMD:C_0402_1005Metric"
 			(at 264.16 56.1848 0)
 			(effects
@@
 			)
 		)
-		(property "MPN" "C161494"
+		(property "MPN" "C106204"
 			(at 260.35 57.15 0)
 			(effects
@@
 			)
 		)
-		(property "Footprint" "Resistor_SMD:R_0201_0603Metric"
+		(property "Footprint" "Resistor_SMD:R_0402_1005Metric"
 			(at 151.892 74.93 90)
 			(effects
@@
 			)
 		)
-		(property "MPN" "C490808"
+		(property "MPN" "C25744"
 			(at 153.67 74.93 0)
 			(effects
@@
 			)
 		)
-		(property "Footprint" "Capacitor_SMD:C_0201_0603Metric"
+		(property "Footprint" "Capacitor_SMD:C_0402_1005Metric"
 			(at 264.16 46.0248 0)
 			(effects
@@
 			)
 		)
-		(property "MPN" "C76933"
+		(property "MPN" "C326606"
 			(at 260.35 46.99 0)
 			(effects
@@
 		)
 		(instances
-			(project ""
+			(project "drehm-fc"
 				(path "/78677983-3e2d-46c3-90bf-4f512dd2e99e"
 					(reference "#FLG02")
@@
 		)
 		(instances
-			(project ""
+			(project "drehm-fc"
 				(path "/78677983-3e2d-46c3-90bf-4f512dd2e99e"
 					(reference "#PWR015")
@@
 		)
 		(instances
-			(project ""
+			(project "drehm-fc"
 				(path "/78677983-3e2d-46c3-90bf-4f512dd2e99e"
 					(reference "#FLG03")
@@
 		)
 		(instances
-			(project ""
+			(project "drehm-fc"
 				(path "/78677983-3e2d-46c3-90bf-4f512dd2e99e"
 					(reference "#PWR016")
